File: PCB/Remote/Remote.kicad_sch (KiCad schematic)
At the start: 71 parts, among them J1 LCD, J2 DC, J3 TEMP, J4 LCD, J5 Reset, J6 USB-C-Socket-H, J7 TC2030-USB-NL-DS, T1 T3902_MEMS_Mic, U1 ESP32-S3-MINI-1, U2 SCD41, U3 MD8942, U4 TMP1075DSG, U5 GZP6816D, U7 SHT40, U8 VEML6040

Commit message: New rendere
Parts:
- added C13: 4.7uF, RevK:C_0402, symbol Device:C
- added D10, D11, D12, D13, D14, D3, D7, D8, D9: ~, RevK:DFN1006-2L, symbol RevK:ES05D1MC10
- added R9: 100R, RevK:R_0402, symbol Device:R
- added TP21, TP23, TP24, TP26: TestPoint, RevK:TestPad, symbol Connector:TestPoint
- added TP22, TP25: TestPoint, RevK:TestPadSquare, symbol Connector:TestPoint
- added U6: IRM-H638T/TR2, RevK:SMD-4P,4x5mm, symbol RevK:IRM-H638T/TR2
- R6, R7: value 10K -> 4k7; MPN C25744 -> C25900
Connections:
- net +3.3V: now also R9.2, TP23.1, TP26.1
- net E: now also D9.1
- net GND: now also C13.2, D10.2, D11.1, D12.1, D13.1, D14.1, D3.2, D7.2, D8.2, D9.2, TP22.1, TP25.1, U6.1 (GND), U6.2 (GND)
- net N: now also D7.1
- net P: now also D3.1
- net S: now also D8.1
- net SCL: now also D13.2
- net SDA: now also D14.2
- net TEMP: now also D11.2
- net W: now also D10.1
- net IR: now reaches U1.22 (GPIO18)
- net IR: now also D12.2, TP21.1, TP24.1, U6.3 (OUT)
- new net: C13.1, R9.1, U6.4 (VCC)
- no-connect marks 21 -> 20

Commit message: Clean up BOM
Parts:
- C13: MPN C194427 -> C23733
- R9: MPN (none) -> C25076
- TP1, TP10, TP11, TP12, TP13, TP14, TP15, TP16, TP17, TP18, TP19, TP2, TP20, TP21, TP22, TP23, TP24, TP25, TP26, TP3, TP4, TP5, TP6, TP7, TP8, TP9: now left out of the parts list
Changed lines of the file:
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@@
 		(unit 1)
 		(exclude_from_sim no)
-		(in_bom yes)
+		(in_bom no)
 		(on_board yes)
 		(dnp no)
@@
 		(unit 1)
 		(exclude_from_sim no)
-		(in_bom yes)
+		(in_bom no)
 		(on_board yes)
 		(dnp no)
@@
 		(unit 1)
 		(exclude_from_sim no)
-		(in_bom yes)
+		(in_bom no)
 		(on_board yes)
 		(dnp no)
@@
 		(unit 1)
 		(exclude_from_sim no)
-		(in_bom yes)
+		(in_bom no)
 		(on_board yes)
 		(dnp no)
@@
 		(unit 1)
 		(exclude_from_sim no)
-		(in_bom yes)
+		(in_bom no)
 		(on_board yes)
 		(dnp no)
@@
 		(unit 1)
 		(exclude_from_sim no)
-		(in_bom yes)
+		(in_bom no)
 		(on_board yes)
 		(dnp no)
@@
 		(unit 1)
 		(exclude_from_sim no)
-		(in_bom yes)
+		(in_bom no)
 		(on_board yes)
 		(dnp no)
@@
 		(unit 1)
 		(exclude_from_sim no)
-		(in_bom yes)
+		(in_bom no)
 		(on_board yes)
 		(dnp no)
@@
 		(unit 1)
 		(exclude_from_sim no)
-		(in_bom yes)
+		(in_bom no)
 		(on_board yes)
 		(dnp no)
@@
 			)
 		)
-		(property "MPN" "C194427"
+		(property "MPN" "C23733"
 			(at 183.515 114.935 0)
 			(effects
@@
 		(unit 1)
 		(exclude_from_sim no)
-		(in_bom yes)
+		(in_bom no)
 		(on_board yes)
 		(dnp no)
@@
 		(unit 1)
 		(exclude_from_sim no)
-		(in_bom yes)
+		(in_bom no)
 		(on_board yes)
 		(dnp no)
@@
 		(unit 1)
 		(exclude_from_sim no)
-		(in_bom yes)
+		(in_bom no)
 		(on_board yes)
 		(dnp no)
@@
 			)
 		)
+		(property "MPN" "C25076"
+			(at 187.325 109.855 90)
+			(effects
+				(font
+					(size 1.27 1.27)
+				)
+				(hide yes)
+			)
+		)
 		(pin "1"
 		)
@@
 		(unit 1)
 		(exclude_from_sim no)
-		(in_bom yes)
+		(in_bom no)
 		(on_board yes)
 		(dnp no)
@@
 		(unit 1)
 		(exclude_from_sim no)
-		(in_bom yes)
+		(in_bom no)
 		(on_board yes)
 		(dnp no)
@@
 		(unit 1)
 		(exclude_from_sim no)
-		(in_bom yes)
+		(in_bom no)
 		(on_board yes)
 		(dnp no)
@@
 		(unit 1)
 		(exclude_from_sim no)
-		(in_bom yes)
+		(in_bom no)
 		(on_board yes)
 		(dnp no)
@@
 		(unit 1)
 		(exclude_from_sim no)
-		(in_bom yes)
+		(in_bom no)
 		(on_board yes)
 		(dnp no)
@@
 		(unit 1)
 		(exclude_from_sim no)
-		(in_bom yes)
+		(in_bom no)
 		(on_board yes)
 		(dnp no)
@@
 		(unit 1)
 		(exclude_from_sim no)
-		(in_bom yes)
+		(in_bom no)
 		(on_board yes)
 		(dnp no)
@@
 		(unit 1)
 		(exclude_from_sim no)
-		(in_bom yes)
+		(in_bom no)
 		(on_board yes)
 		(dnp no)
@@
 		(unit 1)
 		(exclude_from_sim no)
-		(in_bom yes)
+		(in_bom no)
 		(on_board yes)
 		(dnp no)
@@
 		(unit 1)
 		(exclude_from_sim no)
-		(in_bom yes)
+		(in_bom no)
 		(on_board yes)
 		(dnp no)
@@
 		(unit 1)
 		(exclude_from_sim no)
-		(in_bom yes)
+		(in_bom no)
 		(on_board yes)
 		(dnp no)
@@
 		(unit 1)
 		(exclude_from_sim no)
-		(in_bom yes)
+		(in_bom no)
 		(on_board yes)
 		(dnp no)
@@
 		(unit 1)
 		(exclude_from_sim no)
-		(in_bom yes)
+		(in_bom no)
 		(on_board yes)
 		(dnp no)
@@
 		(unit 1)
 		(exclude_from_sim no)
-		(in_bom yes)
+		(in_bom no)
 		(on_board yes)
 		(dnp no)

Commit message: Re render/case
Other:
- note added: "I2C addresses (hex) 10 VEML6040 18 MCP9808 78 GZP6816D 62 SCD41 15 T6793 48 TMP1075 44 SHT40 76 BME488"
- note removed: "I2C addresses (hex) 10 VEML6040 18 MCP9808 78 GZP6816D 62 SCD41 15 T6793 48 TMP1075 44 SHT40"
Changed lines of the file:
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@@
 		(comment 2 "www.me.uk")
 	)
-	(text "I2C addresses (hex)\n10 VEML6040\n18 MCP9808\n78 GZP6816D\n62 SCD41\n15 T6793\n48 TMP1075\n44 SHT40"
+	(text "I2C addresses (hex)\n10 VEML6040\n18 MCP9808\n78 GZP6816D\n62 SCD41\n15 T6793\n48 TMP1075\n44 SHT40\n76 BME488"
 		(exclude_from_sim no)
 		(at 22.098 80.772 0)

Commit message: Library update
Parts:
- removed TP22, TP25: TestPoint, RevK:TestPadSquare, symbol Connector:TestPoint
- removed TP23, TP26: TestPoint, RevK:TestPad, symbol Connector:TestPoint
- removed U6: IRM-H638T/TR2, RevK:SMD-4P,4x5mm, symbol RevK:IRM-H638T/TR2
- added U6: IRMHF384, RevK:IR-SMD-4P,3.35x3.9mm, symbol RevK:IRMHF384
- C13: value 4.7uF -> 47uF; footprint RevK:C_0402 -> RevK:C_0603; MPN C23733 -> (none)
- R9: value 100R -> 47R; MPN C25076 -> C25118
Connections:
- net GND: now also U6.3 (GND), U6.4 (GND)
- net IR: now also U6.1 (OUT)
- net at C13.1, R9.1: now also U6.2 (VCC)
Other:
- moved on the sheet: D12

Commit message: Library update
Parts:
- D4, D6: footprint RevK:SMD1010-Side -> RevK:SMD1010-Side2
Changed lines of the file:
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@@
 			)
 		)
-		(property "Footprint" "RevK:SMD1010-Side"
+		(property "Footprint" "RevK:SMD1010-Side2"
 			(at 147.32 22.225 0)
 			(effects
@@
 			)
 		)
-		(property "Footprint" "RevK:SMD1010-Side"
+		(property "Footprint" "RevK:SMD1010-Side2"
 			(at 162.56 22.225 0)
 			(effects

Commit message: Library update
Parts:
- U7: footprint RevK:Sensirion_DFN-4_1.5x1.5mm_P0.5mm_SHT4x -> RevK:Sensirion_DFN-4_1.5x1.5mm_P0.5mm_SHT4x-Side
Changed lines of the file:
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@@
 			)
 		)
-		(property "Footprint" "RevK:Sensirion_DFN-4_1.5x1.5mm_P0.5mm_SHT4x"
+		(property "Footprint" "RevK:Sensirion_DFN-4_1.5x1.5mm_P0.5mm_SHT4x-Side"
 			(at 254.635 145.415 0)
 			(effects

Commit message: New layout - IR back to sensible place
Parts:
- added TP22, TP25: TestPoint, RevK:TestPadSquare, symbol Connector:TestPoint
- added TP23, TP26: TestPoint, RevK:TestPad, symbol Connector:TestPoint
- D5: footprint RevK:SMD1010-Side -> RevK:SMD1010-Side2
Connections:
- net +3.3V: now also TP23.1, TP26.1
- net GND: now also TP22.1, TP25.1

Commit message: Moved mic
Parts:
- T1: footprint RevK:T3902_MEMS_Mic -> RevK:T3902_MEMS_Mic-Open
Connections:
- net MCLK: now also U1.29 (GPIO34); no longer U1.14 (GPIO10)
- net MDATA: now also U1.28 (GPIO33); no longer U1.15 (GPIO11)
Changed lines of the file:
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@@
 	)
 	(no_connect
-		(at 205.74 59.055)
+		(at 175.26 66.675)
 	)
 	(no_connect
@@
 	)
 	(no_connect
-		(at 205.74 61.595)
+		(at 175.26 69.215)
 	)
 	(no_connect
@@
 	(global_label "MCLK"
 		(shape output)
-		(at 175.26 66.675 180)
+		(at 205.74 61.595 0)
 		(fields_autoplaced yes)
 		(effects
@@
 				(size 1.27 1.27)
 			)
-			(justify right)
+			(justify left)
 		)
 		(property "Intersheetrefs" "${INTERSHEET_REFS}"
-			(at 167.9095 66.675 0)
+			(at 213.0905 61.595 0)
 			(effects
 				(font
 					(size 1.27 1.27)
 				)
-				(justify right)
+				(justify left)
 				(hide yes)
 			)
@@
 	(global_label "MDATA"
 		(shape input)
-		(at 175.26 69.215 180)
+		(at 205.74 59.055 0)
 		(fields_autoplaced yes)
 		(effects
@@
 				(size 1.27 1.27)
 			)
-			(justify right)
+			(justify left)
 		)
 		(property "Intersheetrefs" "${INTERSHEET_REFS}"
-			(at 167.0628 69.215 0)
+			(at 213.9372 59.055 0)
 			(effects
 				(font
 					(size 1.27 1.27)
 				)
-				(justify right)
+				(justify left)
 				(hide yes)
 			)
@@
 			)
 		)
-		(property "Footprint" "RevK:T3902_MEMS_Mic"
+		(property "Footprint" "RevK:T3902_MEMS_Mic-Open"
 			(at 204.851 120.015 0)
 			(effects
