File: PCB/Remote/Remote.kicad_sch (KiCad schematic)
At the start: 89 parts, among them J1 LCD, J2 DC, J3 TEMP, J4 LCD, J5 Reset, J6 USB-C-Socket-H, J7 TC2030-USB-NL-DS, T1 T3902_MEMS_Mic, U1 ESP32-S3-MINI-1, U2 SCD41, U3 MD8942, U4 TMP1075DSG, U5 GZP6816D, U6 IRMHF384, U7 SHT40, U8 VEML6040

Commit message: Library update
Parts:
- removed C2: 22uF, RevK:C_0402, symbol Device:C
- removed C21: 10uF 35V, RevK:C_0603_, symbol RevK:Hidden
- removed C22: 10uF 6.3V, RevK:C_0603_, symbol RevK:Hidden
- removed C23: 100nF, RevK:C_0603_, symbol RevK:Hidden
- removed D19, D20: MBR0530, RevK:D_SOD-123, symbol Diode:1N5819
- removed L4: 10uH, RevK:L_4x4_, symbol RevK:Hidden
- removed R17: 124k, RevK:R_0402_, symbol RevK:Hidden
- removed R18: 39k2, RevK:R_0402_, symbol RevK:Hidden
- removed R27: 1M, RevK:R_0402_, symbol RevK:Hidden
- removed U3: MD8942, RevK:SOT-23-6-MD8942, symbol RevK:MD89420-RegBlock
- added C20: 22uF 25V, RevK:C_0805, symbol Device:C
- added C21: 100nF 25V, RevK:C_0402, symbol Device:C
- added C22, C25: 100nF, RevK:C_0201, symbol Device:C
- added C23: 18pF, RevK:C_0201, symbol Device:C
- added C24: 47uF 6V, RevK:C_0805, symbol Device:C
- added D19, D20: DKS34, RevK:D_SOD-123FL, symbol Device:D_Schottky
- added L2: 4.7uH, RevK:L_5x5, symbol Device:L
- added R10, R11: 150k 1%, RevK:R_0201, symbol Device:R
- added R12: 33k 1%, RevK:R_0201, symbol Device:R
- added U9: TPS562246, RevK:SOT-563, symbol RevK:TPS562246
- C1, C10, C11, C12, C5, C6, C8, C9: footprint RevK:C_0402 -> RevK:C_0201; MPN (none) -> C76934
- C3, C7: footprint RevK:C_0402 -> RevK:C_0201
- R13, R6, R7: footprint RevK:R_0402 -> RevK:R_0201; MPN C25900 -> C7467262
- R3, R4: footprint RevK:R_0402 -> RevK:R_0201; MPN C25905 -> C473460
- R5: footprint RevK:R_0402 -> RevK:R_0201; MPN C25744 -> C102690
- R9: MPN C25118 -> C854484
Connections:
- net +3.3V: now also C1.2, C10.2, C11.2, C12.2, C5.2, C6.2, C8.2, C9.2, C23.2, C24.1, C25.2, L2.2, R11.1; no longer C1.1, C10.1, C11.1, C12.1, C5.1, C6.1, C8.1, C9.1
- net GND: now also C1.1, C10.1, C11.1, C12.1, C5.1, C6.1, C8.1, C9.1, C20.2, C21.2, C24.2, C25.1, R12.2, U9.3 (GND); no longer C1.2, C10.2, C11.2, C12.2, C5.2, C6.2, C8.2, C9.2
- net VBUS: now also D20.2 (A)
- net VDC: now also C20.1, C21.1, D19.1 (K), D20.1 (K), R10.2, U9.1 (VIN)
- net at J2.2 (DC): now also D19.2 (A)
- new net BST: C22.1, U9.4 (VBST)
- new net EN: R10.1, U9.5 (EN)
- new net FB: C23.1, R11.2, R12.1, U9.6 (VFB)
- new net SW: C22.2, L2.1, U9.2 (SW)
- no-connect marks 20 -> 19
Other:
- note added: "2A 3.3V power block"
- moved on the sheet: C13, C3, C4, D4, D5, D6, J2, J5, R5, R9, U1, U6

Commit message: New LED
Parts:
- D4, D5, D6: footprint RevK:SMD1010-Side2 -> RevK:SMD1615; symbol RevK:WS2812B-1mm -> RevK:WS2812B-1.5mm; MPN C5349953 -> C5349954
Connections:
- net +3.3V: now also D4.3 (+), D5.3 (+), D6.3 (+); no longer D4.2 (+), D5.2 (+), D6.2 (+)
- net GND: now also D4.1 (-), D5.1 (-), D6.1 (-); no longer D4.3 (-), D5.3 (-), D6.3 (-)
- net LED: now also D4.2 (I); no longer D4.4 (I)
- net at D5.4 (O): now also D6.2 (I); no longer D4.1 (O)
- net at D6.4 (O): no longer D5.1 (O)
- new net: D4.4 (O), D5.2 (I)
Changed lines of the file:
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@@
 	)
 	(symbol
-		(lib_id "RevK:WS2812B-1mm")
+		(lib_id "RevK:WS2812B-1.5mm")
 		(at 83.185 139.7 0)
-		(mirror x)
 		(unit 1)
 		(exclude_from_sim no)
@@
 		)
 		(property "Value" "XL-1010RGBC-WS2812B"
-			(at 84.455 133.985 0)
+			(at 84.455 145.415 0)
 			(effects
 				(font
@@
 			)
 		)
-		(property "Footprint" "RevK:SMD1010-Side2"
+		(property "Footprint" "RevK:SMD1615"
 			(at 84.455 132.08 0)
 			(effects
@@
 			)
 		)
-		(property "Datasheet" "https://datasheet.lcsc.com/lcsc/2301111010_XINGLIGHT-XL-1010RGBC-WS2812B_C5349953.pdf"
+		(property "Datasheet" "https://www.lcsc.com/datasheet/C5349954.pdf"
 			(at 84.455 130.175 0)
 			(effects
@@
 			)
 		)
-		(property "MPN" "C5349953"
+		(property "MPN" "C5349954"
 			(at 84.455 128.27 0)
 			(effects
@@
 	)
 	(symbol
-		(lib_id "RevK:WS2812B-1mm")
+		(lib_id "RevK:WS2812B-1.5mm")
 		(at 98.425 139.7 0)
-		(mirror x)
 		(unit 1)
 		(exclude_from_sim no)
@@
 		)
 		(property "Value" "XL-1010RGBC-WS2812B"
-			(at 99.695 133.985 0)
+			(at 99.695 145.415 0)
 			(effects
 				(font
@@
 			)
 		)
-		(property "Footprint" "RevK:SMD1010-Side2"
+		(property "Footprint" "RevK:SMD1615"
 			(at 99.695 132.08 0)
 			(effects
@@
 			)
 		)
-		(property "Datasheet" "https://datasheet.lcsc.com/lcsc/2301111010_XINGLIGHT-XL-1010RGBC-WS2812B_C5349953.pdf"
+		(property "Datasheet" "https://www.lcsc.com/datasheet/C5349954.pdf"
 			(at 99.695 130.175 0)
 			(effects
@@
 			)
 		)
-		(property "MPN" "C5349953"
+		(property "MPN" "C5349954"
 			(at 99.695 128.27 0)
 			(effects
@@
 	)
 	(symbol
-		(lib_id "RevK:WS2812B-1mm")
+		(lib_id "RevK:WS2812B-1.5mm")
 		(at 90.805 139.7 0)
-		(mirror x)
 		(unit 1)
 		(exclude_from_sim no)
@@
 		)
 		(property "Value" "XL-1010RGBC-WS2812B"
-			(at 92.075 133.985 0)
+			(at 92.075 145.415 0)
 			(effects
 				(font
@@
 			)
 		)
-		(property "Footprint" "RevK:SMD1010-Side2"
+		(property "Footprint" "RevK:SMD1615"
 			(at 92.075 132.08 0)
 			(effects
@@
 			)
 		)
-		(property "Datasheet" "https://datasheet.lcsc.com/lcsc/2301111010_XINGLIGHT-XL-1010RGBC-WS2812B_C5349953.pdf"
+		(property "Datasheet" "https://www.lcsc.com/datasheet/C5349954.pdf"
 			(at 92.075 130.175 0)
 			(effects
@@
 			)
 		)
-		(property "MPN" "C5349953"
+		(property "MPN" "C5349954"
 			(at 92.075 128.27 0)
 			(effects

Commit message: Tweaks, but cases look wrong
Parts:
- U9: footprint RevK:SOT-563 -> RevK:SOT-5x3-6
Changed lines of the file:
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@@
 			)
 		)
+		(property "Sim.Enable" "0"
+			(at 273.685 173.355 0)
+			(effects
+				(font
+					(size 1.27 1.27)
+				)
+				(hide yes)
+			)
+		)
 		(instances
 			(project "EnvMon"
@@
 	)
 	(symbol
-		(lib_id "power:PWR_FLAG")
-		(at 120.65 37.465 270)
-		(unit 1)
-		(exclude_from_sim no)
-		(in_bom yes)
-		(on_board yes)
-		(dnp no)
-		(fields_autoplaced yes)
-		(property "Reference" "#FLG02"
-			(at 122.555 37.465 0)
-			(effects
-				(font
-					(size 1.27 1.27)
-				)
-				(hide yes)
-			)
-		)
-		(property "Value" "PWR_FLAG"
-			(at 123.825 37.465 90)
-			(effects
-				(font
-					(size 1.27 1.27)
-				)
-				(justify left)
-			)
-		)
-		(property "Footprint" ""
-			(at 120.65 37.465 0)
-			(effects
-				(font
-					(size 1.27 1.27)
-				)
-				(hide yes)
-			)
-		)
-		(property "Datasheet" "~"
-			(at 120.65 37.465 0)
-			(effects
-				(font
-					(size 1.27 1.27)
-				)
-				(hide yes)
-			)
-		)
-		(property "Description" "Special symbol for telling ERC where power comes from"
-			(at 120.65 37.465 0)
-			(effects
-				(font
-					(size 1.27 1.27)
-				)
-				(hide yes)
-			)
-		)
-		(pin "1"
-		)
-		(instances
-			(project "EnvMon"
-				(path "/12422a89-3d0c-485c-9386-f77121fd68fd"
-					(reference "#FLG02")
-					(unit 1)
-				)
-			)
-		)
-	)
-	(symbol
 		(lib_id "RevK:ES05D1MC10")
 		(at 88.9 109.855 0)
@@
 			)
 		)
+		(property "Sim.Enable" "0"
+			(at 276.86 176.53 0)
+			(effects
+				(font
+					(size 1.27 1.27)
+				)
+				(hide yes)
+			)
+		)
 		(instances
 			(project "EnvMon"
@@
 			)
 		)
-		(property "Footprint" "RevK:SOT-563"
+		(property "Footprint" "RevK:SOT-5x3-6"
 			(at 223.52 27.305 0)
 			(effects
@@
 	)
 	(symbol
-		(lib_name "TC2030-USB-NL_1")
 		(lib_id "RevK:TC2030-USB-NL")
 		(at 121.285 82.55 0)
@@
 			)
 		)
+		(property "Sim.Enable" "0"
+			(at 280.035 173.355 0)
+			(effects
+				(font
+					(size 1.27 1.27)
+				)
+				(hide yes)
+			)
+		)
 		(instances
 			(project "EnvMon"
@@
 	)
 	(symbol
+		(lib_id "power:PWR_FLAG")
+		(at 174.625 111.76 0)
+		(unit 1)
+		(exclude_from_sim no)
+		(in_bom yes)
+		(on_board yes)
+		(dnp no)
+		(fields_autoplaced yes)
+		(property "Reference" "#FLG02"
+			(at 174.625 109.855 0)
+			(effects
+				(font
+					(size 1.27 1.27)
+				)
+				(hide yes)
+			)
+		)
+		(property "Value" "PWR_FLAG"
+			(at 174.625 107.6269 0)
+			(effects
+				(font
+					(size 1.27 1.27)
+				)
+			)
+		)
+		(property "Footprint" ""
+			(at 174.625 111.76 0)
+			(effects
+				(font
+					(size 1.27 1.27)
+				)
+				(hide yes)
+			)
+		)
+		(property "Datasheet" "~"
+			(at 174.625 111.76 0)
+			(effects
+				(font
+					(size 1.27 1.27)
+				)
+				(hide yes)
+			)
+		)
+		(property "Description" "Special symbol for telling ERC where power comes from"
+			(at 174.625 111.76 0)
+			(effects
+				(font
+					(size 1.27 1.27)
+				)
+				(hide yes)
+			)
+		)
+		(pin "1"
+		)
+		(instances
+			(project ""
+				(path "/12422a89-3d0c-485c-9386-f77121fd68fd"
+					(reference "#FLG02")
+					(unit 1)
+				)
+			)
+		)
+	)
+	(symbol
 		(lib_id "power:GND")
 		(at 121.285 175.895 0)
@@
 	)
 	(symbol
-		(lib_id "power:GND")
-		(at 120.65 37.465 270)
-		(unit 1)
-		(exclude_from_sim no)
-		(in_bom yes)
-		(on_board yes)
-		(dnp no)
-		(property "Reference" "#PWR021"
-			(at 114.3 37.465 0)
-			(effects
-				(font
-					(size 1.27 1.27)
-				)
-				(hide yes)
-			)
-		)
-		(property "Value" "GND"
-			(at 116.078 37.465 90)
-			(effects
-				(font
-					(size 1.27 1.27)
-				)
-			)
-		)
-		(property "Footprint" ""
-			(at 120.65 37.465 0)
-			(effects
-				(font
-					(size 1.27 1.27)
-				)
-				(hide yes)
-			)
-		)
-		(property "Datasheet" ""
-			(at 120.65 37.465 0)
-			(effects
-				(font
-					(size 1.27 1.27)
-				)
-				(hide yes)
-			)
-		)
-		(property "Description" "Power symbol creates a global label with name \"GND\" , ground"
-			(at 120.65 37.465 0)
-			(effects
-				(font
-					(size 1.27 1.27)
-				)
-				(hide yes)
-			)
-		)
-		(pin "1"
-		)
-		(instances
-			(project "EnvMon"
-				(path "/12422a89-3d0c-485c-9386-f77121fd68fd"
-					(reference "#PWR021")
-					(unit 1)
-				)
-			)
-		)
-	)
-	(symbol
 		(lib_id "power:+3.3V")
 		(at 121.285 158.115 0)
@@
 			(at 276.86 170.18 0)
 			(effects
+				(font
+					(size 1.27 1.27)
+				)
+				(hide yes)
+			)
+		)
+		(property "Sim.Enable" "0"
+			(at 276.86 170.18 0)
+			(effects

Commit message: Library update
Parts:
- D4: value XL-1010RGBC-WS2812B -> XL-1615RGBC-2812B; footprint RevK:SMD1615 -> RevK:SMD1615-Side
- D5, D6: footprint RevK:SMD1615 -> RevK:SMD1615-Side
Changed lines of the file:
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@@
 			)
 		)
-		(property "Sim.Enable" "0"
-			(at 273.685 173.355 0)
-			(effects
-				(font
-					(size 1.27 1.27)
-				)
-				(hide yes)
-			)
-		)
 		(instances
 			(project "EnvMon"
@@
 			)
 		)
-		(property "Value" "XL-1010RGBC-WS2812B"
+		(property "Value" "XL-1615RGBC-2812B"
 			(at 84.455 145.415 0)
 			(effects
@@
 			)
 		)
-		(property "Footprint" "RevK:SMD1615"
+		(property "Footprint" "RevK:SMD1615-Side"
 			(at 84.455 132.08 0)
 			(effects
@@
 			)
 		)
-		(property "Sim.Enable" "0"
-			(at 276.86 176.53 0)
-			(effects
-				(font
-					(size 1.27 1.27)
-				)
-				(hide yes)
-			)
-		)
 		(instances
 			(project "EnvMon"
@@
 			)
 		)
-		(property "Footprint" "RevK:SMD1615"
+		(property "Footprint" "RevK:SMD1615-Side"
 			(at 99.695 132.08 0)
 			(effects
@@
 			)
 		)
-		(property "Sim.Enable" "0"
-			(at 280.035 173.355 0)
-			(effects
-				(font
-					(size 1.27 1.27)
-				)
-				(hide yes)
-			)
-		)
 		(instances
 			(project "EnvMon"
@@
 			)
 		)
-		(property "Footprint" "RevK:SMD1615"
+		(property "Footprint" "RevK:SMD1615-Side"
 			(at 92.075 132.08 0)
 			(effects
@@
 			(at 276.86 170.18 0)
 			(effects
-				(font
-					(size 1.27 1.27)
-				)
-				(hide yes)
-			)
-		)
-		(property "Sim.Enable" "0"
-			(at 276.86 170.18 0)
-			(effects
