File: PCB/RemoteDev/Remote.kicad_sch (KiCad schematic)
At the start: 91 parts, among them J1 LCD, J2 DC, J3 TEMP, J4 LCD, J5 Reset, J6 USB-C-Socket-H, J7 TC2030-USB-NL-DS, T1 T3902_MEMS_Mic, U1 ESP32-S3-MINI-1, U2 SCD41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

Commit message: Latest renders
Parts:
- R9: footprint RevK:R_0402 -> RevK:R_0201; MPN C25118 -> (none)
Changed lines of the file:
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@@
 			)
 		)
-		(property "Footprint" "RevK:R_0402"
+		(property "Footprint" "RevK:R_0201"
 			(at 181.61 113.538 90)
 			(effects
@@
 			)
 		)
-		(property "MPN" "C25118"
+		(property "MPN" ""
 			(at 181.61 111.76 90)
 			(effects

Commit message: wider
Parts:
- removed D19, D20: MBR0530, RevK:D_SOD-123, symbol Diode:1N5819
- added D19, D20: DKS22, RevK:D_SOD-123FL, symbol Device:D_Schottky
Connections:
- net VBUS: now also D20.2 (A)
- net VDC: now also D19.1 (K), D20.1 (K)
- net at J2.2 (DC): now also D19.2 (A)
Other:
- moved on the sheet: J2
Changed lines of the file:
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@@
 	(wire
 		(pts
+			(xy 266.7 48.26) (xy 265.43 48.26)
+		)
+		(stroke
+			(width 0)
+			(type default)
+		)
+	)
+	(wire
+		(pts
 			(xy 216.535 131.445) (xy 205.105 131.445)
 		)
@@
 	(symbol
 		(lib_id "RevK:PowerIn")
-		(at 270.51 48.26 0)
+		(at 271.78 48.26 0)
 		(unit 1)
 		(exclude_from_sim no)
@@
 		(dnp no)
 		(property "Reference" "J2"
-			(at 271.78 45.72 0)
+			(at 273.05 45.72 0)
 			(effects
 				(font
@@
 		)
 		(property "Value" "DC"
-			(at 280.67 48.895 0)
+			(at 281.94 48.895 0)
 			(effects
 				(font
@@
 		)
 		(property "Footprint" "RevK:WAGO-2060-452-998-404"
-			(at 270.51 48.26 0)
+			(at 271.78 48.26 0)
 			(effects
 				(font
@@
 		)
 		(property "Datasheet" "~"
-			(at 270.51 48.26 0)
+			(at 271.78 48.26 0)
 			(effects
 				(font
@@
 		)
 		(property "Description" ""
-			(at 270.51 48.26 0)
+			(at 271.78 48.26 0)
 			(effects
 				(font
@@
 		)
 		(property "MPN" "C2765055"
-			(at 270.51 48.26 0)
+			(at 271.78 48.26 0)
 			(effects
 				(font
@@
 	)
 	(symbol
-		(lib_id "Diode:1N5819")
-		(at 261.62 50.8 0)
-		(unit 1)
-		(exclude_from_sim no)
-		(in_bom yes)
-		(on_board yes)
-		(dnp no)
-		(property "Reference" "D19"
-			(at 260.35 53.34 0)
-			(effects
-				(font
-					(size 1.27 1.27)
-				)
-			)
-		)
-		(property "Value" "MBR0530"
-			(at 257.175 55.245 0)
-			(effects
-				(font
-					(size 1.27 1.27)
-				)
-			)
-		)
-		(property "Footprint" "RevK:D_SOD-123"
-			(at 261.62 55.245 0)
-			(effects
-				(font
-					(size 1.27 1.27)
-				)
-				(hide yes)
-			)
-		)
-		(property "Datasheet" ""
-			(at 261.62 50.8 0)
-			(effects
-				(font
-					(size 1.27 1.27)
-				)
-				(hide yes)
-			)
-		)
-		(property "Description" ""
-			(at 261.62 50.8 0)
-			(effects
-				(font
-					(size 1.27 1.27)
-				)
-				(hide yes)
-			)
-		)
-		(property "MPN" "C5204746"
-			(at 261.62 50.8 0)
-			(effects
-				(font
-					(size 1.27 1.27)
-				)
-				(hide yes)
-			)
-		)
-		(pin "1"
-		)
-		(pin "2"
-		)
-		(instances
-			(project "EnvMon"
-				(path "/12422a89-3d0c-485c-9386-f77121fd68fd"
-					(reference "D19")
-					(unit 1)
-				)
-			)
-		)
-	)
-	(symbol
 		(lib_id "Connector:TestPoint")
 		(at 220.345 163.83 90)
@@
 	(symbol
 		(lib_id "power:VDC")
-		(at 257.81 50.8 90)
+		(at 259.08 50.8 90)
 		(unit 1)
 		(exclude_from_sim no)
@@
 		(fields_autoplaced yes)
 		(property "Reference" "#PWR04"
-			(at 261.62 50.8 0)
+			(at 262.89 50.8 0)
 			(effects
 				(font
@@
 		)
 		(property "Value" "VDC"
-			(at 254.635 50.8 90)
+			(at 255.905 50.8 90)
 			(effects
 				(font
@@
 		)
 		(property "Footprint" ""
-			(at 257.81 50.8 0)
+			(at 259.08 50.8 0)
 			(effects
 				(font
@@
 		)
 		(property "Datasheet" ""
-			(at 257.81 50.8 0)
+			(at 259.08 50.8 0)
 			(effects
 				(font
@@
 		)
 		(property "Description" "Power symbol creates a global label with name \"VDC\""
-			(at 257.81 50.8 0)
+			(at 259.08 50.8 0)
 			(effects
 				(font
@@
 	)
 	(symbol
-		(lib_id "Diode:1N5819")
-		(at 261.62 61.595 0)
-		(unit 1)
-		(exclude_from_sim no)
-		(in_bom yes)
-		(on_board yes)
-		(dnp no)
-		(property "Reference" "D20"
-			(at 260.35 64.135 0)
-			(effects
-				(font
-					(size 1.27 1.27)
-				)
-			)
-		)
-		(property "Value" "MBR0530"
-			(at 257.175 66.04 0)
-			(effects
-				(font
-					(size 1.27 1.27)
-				)
-			)
-		)
-		(property "Footprint" "RevK:D_SOD-123"
-			(at 261.62 66.04 0)
-			(effects
-				(font
-					(size 1.27 1.27)
-				)
-				(hide yes)
-			)
-		)
-		(property "Datasheet" ""
-			(at 261.62 61.595 0)
-			(effects
-				(font
-					(size 1.27 1.27)
-				)
-				(hide yes)
-			)
-		)
-		(property "Description" ""
-			(at 261.62 61.595 0)
-			(effects
-				(font
-					(size 1.27 1.27)
-				)
-				(hide yes)
-			)
-		)
-		(property "MPN" "C5204746"
-			(at 261.62 61.595 0)
-			(effects
-				(font
-					(size 1.27 1.27)
-				)
-				(hide yes)
-			)
-		)
-		(pin "1"
-		)
-		(pin "2"
-		)
-		(instances
-			(project "EnvMon"
-				(path "/12422a89-3d0c-485c-9386-f77121fd68fd"
-					(reference "D20")
-					(unit 1)
-				)
-			)
-		)
-	)
-	(symbol
 		(lib_id "RevK:SCD41")
 		(at 157.48 139.065 0)
@@
 					(unit 1)
 				)
+			)
+		)
+	)
+	(symbol
+		(lib_id "Device:D_Schottky")
+		(at 262.89 50.8 0)
+		(unit 1)
+		(exclude_from_sim no)
+		(in_bom yes)
+		(on_board yes)
+		(dnp no)
+		(property "Reference" "D19"
+			(at 262.509 53.34 0)
+			(effects
+				(font
+					(size 1.27 1.27)
+				)
+			)
+		)
+		(property "Value" "DKS22"
+			(at 262.509 55.7643 0)
+			(effects
+				(font
+					(size 1.27 1.27)
+				)
+			)
+		)
+		(property "Footprint" "RevK:D_SOD-123FL"
+			(at 262.89 50.8 0)
+			(effects
+				(font
+					(size 1.27 1.27)
+				)
+				(hide yes)
+			)
+		)
+		(property "Datasheet" "~"
+			(at 262.89 50.8 0)
+			(effects
+				(font
+					(size 1.27 1.27)
+				)
+				(hide yes)
+			)
+		)
+		(property "Description" "Schottky diode"
+			(at 262.89 50.8 0)
+			(effects
+				(font
+					(size 1.27 1.27)
+				)
+				(hide yes)
+			)
+		)
+		(property "MPN" "C727072"
+			(at 262.89 50.8 0)
+			(effects
+				(font
+					(size 1.27 1.27)
+				)
+				(hide yes)
+			)
+		)
+		(pin "2"
+		)
+		(pin "1"
+		)
+		(instances
+			(project "Remote"
+				(path "/12422a89-3d0c-485c-9386-f77121fd68fd"
+					(reference "D19")
+					(unit 1)
+				)
+			)
+		)
+	)
+	(symbol
+		(lib_id "Device:D_Schottky")
+		(at 261.62 61.595 0)
+		(unit 1)
+		(exclude_from_sim no)
+		(in_bom yes)
+		(on_board yes)
+		(dnp no)
+		(property "Reference" "D20"
+			(at 261.239 64.135 0)
+			(effects
+				(font
+					(size 1.27 1.27)
+				)
+			)
+		)
+		(property "Value" "DKS22"
+			(at 261.239 66.5593 0)
+			(effects
+				(font
+					(size 1.27 1.27)
+				)
+			)
+		)
+		(property "Footprint" "RevK:D_SOD-123FL"
+			(at 261.62 61.595 0)
+			(effects
+				(font
+					(size 1.27 1.27)
+				)
+				(hide yes)
+			)
+		)
+		(property "Datasheet" "~"
+			(at 261.62 61.595 0)
+			(effects
+				(font
+					(size 1.27 1.27)
+				)
+				(hide yes)
+			)
+		)
+		(property "Description" "Schottky diode"
+			(at 261.62 61.595 0)
+			(effects
+				(font
+					(size 1.27 1.27)
+				)
+				(hide yes)
+			)
+		)
+		(property "MPN" "C727072"
+			(at 261.62 61.595 0)
+			(effects
+				(font
+					(size 1.27 1.27)
+				)
+				(hide yes)
+			)
+		)
+		(pin "2"
+		)
+		(pin "1"
+		)
+		(instances
+			(project "Remote"
+				(path "/12422a89-3d0c-485c-9386-f77121fd68fd"
+					(reference "D20")
+					(unit 1)
+				)

Commit message: Update reg
Parts:
- U9: symbol RevK:TPS562243 -> RevK:TPS562246; MPN C42295941 -> C41833479
Changed lines of the file:
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@@
 	)
 	(symbol
-		(lib_id "RevK:TPS562243")
+		(lib_id "RevK:TPS562246")
 		(at 222.25 20.955 0)
 		(unit 1)
@@
 			)
 		)
-		(property "Datasheet" "https://www.ti.com/lit/gpn/tps562243"
+		(property "Datasheet" "https://www.ti.com/lit/ds/symlink/tps562246.pdf"
 			(at 222.25 20.955 0)
 			(effects
@@
 			)
 		)
-		(property "MPN" "C42295941"
+		(property "MPN" "C41833479"
 			(at 222.25 20.955 0)
 			(effects

Commit message: Library update
Parts:
- D19, D20: value DKS22 -> DKS34; MPN C727072 -> C727076
- U9: value TPS562243 -> TPS562246
Changed lines of the file:
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@@
 			)
 		)
-		(property "Value" "TPS562243"
+		(property "Value" "TPS562246"
 			(at 222.25 14.1548 0)
 			(effects
@@
 		(dnp no)
 		(property "Reference" "D11"
-			(at 264.414 90.424 0)
+			(at 263.906 96.52 0)
 			(effects
 				(font
@@
 	(symbol
 		(lib_id "power:VBUS")
-		(at 265.43 61.595 270)
+		(at 266.7 57.15 270)
 		(unit 1)
 		(exclude_from_sim no)
@@
 		(fields_autoplaced yes)
 		(property "Reference" "#PWR01"
-			(at 261.62 61.595 0)
+			(at 262.89 57.15 0)
 			(effects
 				(font
@@
 		)
 		(property "Value" "VBUS"
-			(at 268.605 61.595 90)
+			(at 269.875 57.15 90)
 			(effects
 				(font
@@
 		)
 		(property "Footprint" ""
-			(at 265.43 61.595 0)
+			(at 266.7 57.15 0)
 			(effects
 				(font
@@
 		)
 		(property "Datasheet" ""
-			(at 265.43 61.595 0)
+			(at 266.7 57.15 0)
 			(effects
 				(font
@@
 		)
 		(property "Description" "Power symbol creates a global label with name \"VBUS\""
-			(at 265.43 61.595 0)
+			(at 266.7 57.15 0)
 			(effects
 				(font
@@
 	)
 	(symbol
+		(lib_id "Device:D_Schottky")
+		(at 262.89 50.8 0)
+		(unit 1)
+		(exclude_from_sim no)
+		(in_bom yes)
+		(on_board yes)
+		(dnp no)
+		(property "Reference" "D19"
+			(at 259.588 52.07 0)
+			(effects
+				(font
+					(size 1.27 1.27)
+				)
+			)
+		)
+		(property "Value" "DKS34"
+			(at 262.89 53.848 0)
+			(effects
+				(font
+					(size 1.27 1.27)
+				)
+			)
+		)
+		(property "Footprint" "RevK:D_SOD-123FL"
+			(at 262.89 50.8 0)
+			(effects
+				(font
+					(size 1.27 1.27)
+				)
+				(hide yes)
+			)
+		)
+		(property "Datasheet" "~"
+			(at 262.89 50.8 0)
+			(effects
+				(font
+					(size 1.27 1.27)
+				)
+				(hide yes)
+			)
+		)
+		(property "Description" "Schottky diode"
+			(at 262.89 50.8 0)
+			(effects
+				(font
+					(size 1.27 1.27)
+				)
+				(hide yes)
+			)
+		)
+		(property "MPN" "C727076"
+			(at 262.89 50.8 0)
+			(effects
+				(font
+					(size 1.27 1.27)
+				)
+				(hide yes)
+			)
+		)
+		(pin "2"
+		)
+		(pin "1"
+		)
+		(instances
+			(project "Remote"
+				(path "/12422a89-3d0c-485c-9386-f77121fd68fd"
+					(reference "D19")
+					(unit 1)
+				)
+			)
+		)
+	)
+	(symbol
 		(lib_id "Device:R")
 		(at 259.08 29.845 0)
@@
 	(symbol
 		(lib_id "power:VDC")
-		(at 257.81 61.595 90)
+		(at 259.08 57.15 90)
 		(unit 1)
 		(exclude_from_sim no)
@@
 		(fields_autoplaced yes)
 		(property "Reference" "#PWR034"
-			(at 261.62 61.595 0)
+			(at 262.89 57.15 0)
 			(effects
 				(font
@@
 		)
 		(property "Value" "VDC"
-			(at 254.635 61.595 90)
+			(at 255.905 57.15 90)
 			(effects
 				(font
@@
 		)
 		(property "Footprint" ""
-			(at 257.81 61.595 0)
+			(at 259.08 57.15 0)
 			(effects
 				(font
@@
 		)
 		(property "Datasheet" ""
-			(at 257.81 61.595 0)
+			(at 259.08 57.15 0)
 			(effects
 				(font
@@
 		)
 		(property "Description" "Power symbol creates a global label with name \"VDC\""
-			(at 257.81 61.595 0)
+			(at 259.08 57.15 0)
 			(effects
 				(font
@@
 	)
 	(symbol
+		(lib_id "Device:D_Schottky")
+		(at 262.89 57.15 0)
+		(unit 1)
+		(exclude_from_sim no)
+		(in_bom yes)
+		(on_board yes)
+		(dnp no)
+		(property "Reference" "D20"
+			(at 259.588 58.42 0)
+			(effects
+				(font
+					(size 1.27 1.27)
+				)
+			)
+		)
+		(property "Value" "DKS34"
+			(at 262.89 60.198 0)
+			(effects
+				(font
+					(size 1.27 1.27)
+				)
+			)
+		)
+		(property "Footprint" "RevK:D_SOD-123FL"
+			(at 262.89 57.15 0)
+			(effects
+				(font
+					(size 1.27 1.27)
+				)
+				(hide yes)
+			)
+		)
+		(property "Datasheet" "~"
+			(at 262.89 57.15 0)
+			(effects
+				(font
+					(size 1.27 1.27)
+				)
+				(hide yes)
+			)
+		)
+		(property "Description" "Schottky diode"
+			(at 262.89 57.15 0)
+			(effects
+				(font
+					(size 1.27 1.27)
+				)
+				(hide yes)
+			)
+		)
+		(property "MPN" "C727076"
+			(at 262.89 57.15 0)
+			(effects
+				(font
+					(size 1.27 1.27)
+				)
+				(hide yes)
+			)
+		)
+		(pin "2"
+		)
+		(pin "1"
+		)
+		(instances
+			(project "Remote"
+				(path "/12422a89-3d0c-485c-9386-f77121fd68fd"
+					(reference "D20")
+					(unit 1)
+				)
+			)
+		)
+	)
+	(symbol
 		(lib_id "Connector_Generic:Conn_01x02")
 		(at 146.685 100.33 180)
@@
 					(unit 1)
 				)
-			)
-		)
-	)
-	(symbol
-		(lib_id "Device:D_Schottky")
-		(at 262.89 50.8 0)
-		(unit 1)
-		(exclude_from_sim no)
-		(in_bom yes)
-		(on_board yes)
-		(dnp no)
-		(property "Reference" "D19"
-			(at 262.509 53.34 0)
-			(effects
-				(font
-					(size 1.27 1.27)
-				)
-			)
-		)
-		(property "Value" "DKS22"
-			(at 262.509 55.7643 0)
-			(effects
-				(font
-					(size 1.27 1.27)
-				)
-			)
-		)
-		(property "Footprint" "RevK:D_SOD-123FL"
-			(at 262.89 50.8 0)
-			(effects
-				(font
-					(size 1.27 1.27)
-				)
-				(hide yes)
-			)
-		)
-		(property "Datasheet" "~"
-			(at 262.89 50.8 0)
-			(effects
-				(font
-					(size 1.27 1.27)
-				)
-				(hide yes)
-			)
-		)
-		(property "Description" "Schottky diode"
-			(at 262.89 50.8 0)
-			(effects
-				(font
-					(size 1.27 1.27)
-				)
-				(hide yes)
-			)
-		)
-		(property "MPN" "C727072"
-			(at 262.89 50.8 0)
-			(effects
-				(font
-					(size 1.27 1.27)
-				)
-				(hide yes)
-			)
-		)
-		(pin "2"
-		)
-		(pin "1"
-		)
-		(instances
-			(project "Remote"
-				(path "/12422a89-3d0c-485c-9386-f77121fd68fd"
-					(reference "D19")
-					(unit 1)
-				)
-			)
-		)
-	)
-	(symbol
-		(lib_id "Device:D_Schottky")
-		(at 261.62 61.595 0)
-		(unit 1)
-		(exclude_from_sim no)
-		(in_bom yes)
-		(on_board yes)
-		(dnp no)
-		(property "Reference" "D20"
-			(at 261.239 64.135 0)
-			(effects
-				(font
-					(size 1.27 1.27)
-				)
-			)
-		)
-		(property "Value" "DKS22"
-			(at 261.239 66.5593 0)
-			(effects
-				(font
-					(size 1.27 1.27)
-				)
-			)
-		)
-		(property "Footprint" "RevK:D_SOD-123FL"
-			(at 261.62 61.595 0)
-			(effects
-				(font
-					(size 1.27 1.27)
-				)
-				(hide yes)
-			)
-		)
-		(property "Datasheet" "~"
-			(at 261.62 61.595 0)
-			(effects
-				(font
-					(size 1.27 1.27)
-				)
-				(hide yes)
-			)
-		)
-		(property "Description" "Schottky diode"
-			(at 261.62 61.595 0)
-			(effects
-				(font
-					(size 1.27 1.27)
-				)
-				(hide yes)
-			)
-		)
-		(property "MPN" "C727072"
-			(at 261.62 61.595 0)
-			(effects
-				(font
-					(size 1.27 1.27)
-				)
-				(hide yes)
-			)
-		)
-		(pin "2"
-		)
-		(pin "1"
-		)
-		(instances
-			(project "Remote"
-				(path "/12422a89-3d0c-485c-9386-f77121fd68fd"
-					(reference "D20")
-					(unit 1)
-				)

Commit message: MPNs
Parts:
- R13, R6, R7: MPN (none) -> C7467262
- R3, R4: MPN (none) -> C473460
- R5: MPN (none) -> C102690
- R9: footprint RevK:R_0201 -> RevK:R_0402; MPN (none) -> C854484
Changed lines of the file:
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@@
 			)
 		)
-		(property "MPN" ""
+		(property "MPN" "C473460"
 			(at 62.23 35.56 90)
 			(effects
@@
 			)
 		)
-		(property "MPN" ""
+		(property "MPN" "C473460"
 			(at 62.23 33.02 90)
 			(effects
@@
 			)
 		)
-		(property "MPN" ""
+		(property "MPN" "C7467262"
 			(at 236.855 50.165 90)
 			(effects
@@
 			)
 		)
-		(property "MPN" ""
+		(property "MPN" "C7467262"
 			(at 262.255 73.66 90)
 			(effects
@@
 			)
 		)
-		(property "MPN" ""
+		(property "MPN" "C7467262"
 			(at 236.855 56.515 90)
 			(effects
@@
 			)
 		)
-		(property "Footprint" "RevK:R_0201"
+		(property "Footprint" "RevK:R_0402"
 			(at 181.61 113.538 90)
 			(effects
@@
 			)
 		)
-		(property "MPN" ""
+		(property "MPN" "C854484"
 			(at 181.61 111.76 90)
 			(effects
@@
 			)
 		)
-		(property "MPN" ""
+		(property "MPN" "C102690"
 			(at 199.39 97.155 90)
 			(effects

Commit message: Clearing inductror
Parts:
- U9: Rotation Offset -90 -> 180
Changed lines of the file:
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@@
 			)
 		)
-		(property "Rotation Offset" "-90"
+		(property "Rotation Offset" "180"
 			(at 222.25 20.955 0)
 			(effects
